File: Stereo PGA2311 SMD v1,1.brd (EAGLE design)
At the start: 100 x 100 mm, 113 parts, among them K2 351, K3 351, K4 351, K5 351, K6 351, K7 G2R2

Commit message: Add files via upload
Parts:
- C2: device rcl:C0402 -> rcl:C0603
- moved 7805 725.1 mm to (66.0, 48.3)
- moved ATMEGA32 725.1 mm to (15.2, 15.2)
- moved AUDIO-OUT 725.1 mm to (22.9, 51.4)
- moved AUX1 725.1 mm to (90.2, 94.0)
- moved AUX2 725.1 mm to (69.8, 94.0)
- moved AUX3 725.1 mm to (49.5, 94.0)
- moved AUX5 725.1 mm to (8.89, 94.0)
- moved B2 725.1 mm to (63.5, 25.4)
- moved BATTERY 725.1 mm to (48.3, 8.89)
- moved C10 725.1 mm to (86.4, 10.8)
- moved C11 725.1 mm to (86.4, 24.8)
- moved C13 725.1 mm to (86.4, 51.4)
- moved C15 725.1 mm to (73.0, 44.5)
- moved C21 725.1 mm to (40.0, 11.4)
- moved C23 725.1 mm to (30.5, 45.1)
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Other:
- board text removed: "F:/Archiwum/logo2_eagle_my.bmp"
