File: Stereo PGA2311 SMD v1,1.sch (EAGLE design)
At the start: 113 parts, among them K2 351, K3 351, K4 351, K5 351, K6 351, K7 G2R2

Commit message: Add files via upload
Parts:
- C2: device rcl:C-EUC0402 -> rcl:C-EUC0603
Changed lines of the file:
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@@
 <part name="P+3" library="supply1" deviceset="VCC" device=""/>
 <part name="GND3" library="supply1" deviceset="GND" device=""/>
-<part name="C2" library="rcl" deviceset="C-EU" device="C0402" value="100n"/>
+<part name="C2" library="rcl" deviceset="C-EU" device="C0603" value="100n"/>
 <part name="C3" library="rcl" deviceset="C-EU" device="C0603" value="100n"/>
 <part name="GND4" library="supply1" deviceset="GND" device=""/>
